Commit message: Remove Diff drive change robot a bit

File: my_robot/urdf/my_robot.xacro (robot description, xacro)
@@ -3,12 +3,7 @@
   <xacro:include filename="$(find my_robot)/urdf/my_robot.gazebo" />
   <link name="robot_footprint"></link>
-  <joint name="robot_footprint_joint" type="fixed">
-    <origin xyz="0 0 0" rpy="0 0 0" />
-    <parent link="robot_footprint"/>
-    <child link="chassis" />
-  </joint>
   <link name='chassis'>
-    <pose>0 0 0.1 0 0 0</pose>
-    <inertial>
+  <pose>0 0 0.1 0 0 0</pose>
+      <inertial>
       <mass value="15.0"/>
       <origin xyz="0.0 0 0" rpy=" 0 0 0"/>
@@ -17,10 +12,10 @@
           iyy="0.1" iyz="0"
           izz="0.1"
-      />
-    </inertial>
+        />
+      </inertial>
     <collision name='collision'>
       <origin xyz="0 0 0" rpy=" 0 0 0"/>
       <geometry>
-        <box size=".5 .4 .2"/>
+        <box size=".3 .15 .1"/>
       </geometry>
     </collision>
@@ -28,87 +23,136 @@
       <origin xyz="0 0 0" rpy=" 0 0 0"/>
       <geometry>
-        <box size=".5 .4 .2"/>
+        <cylinder radius="0.17" length="0.1"/>
+      </geometry>
+      <material name="blue"/>
+    </visual>
+    <collision name='back_caster_collision'>
+      <origin xyz="-0.1 0 -0.05" rpy=" 0 0 0"/>
+      <geometry>
+        <sphere radius="0.0499"/>
+      </geometry>
+    </collision>
+    <visual name='back_caster_visual'>
+      <origin xyz="-0.1 0 -0.05" rpy=" 0 0 0"/>
+      <geometry>
+        <sphere radius="0.05"/>
+      </geometry>
+    </visual>
+    <collision name='front_caster_collision'>
+      <origin xyz="0.1 0 -0.05" rpy=" 0 0 0"/>
+      <geometry>
+        <sphere radius="0.0499"/>
+      </geometry>
+    </collision>
+    <visual name='front_caster_visual'>
+      <origin xyz="0.1 0 -0.05" rpy=" 0 0 0"/>
+      <geometry>
+        <sphere radius="0.05"/>
       </geometry>
     </visual>
   </link>
-  <link name='front_left_wheel'>
-    <collision>
-      <origin xyz='0 0 0' rpy='-1.57079 0 0'/>
+  <gazebo reference = "chassis">
+    <material> Gazebo/Green </material>
+  </gazebo>
+  <link name="left_wheel">
+  <inertial>
+    <mass value="5.0"/>
+    <origin xyz="0.0 0 0" rpy=" 0 1.5707 1.5707"/>
+    <inertia
+          ixx="0.1" ixy="0" ixz="0"
+          iyy="0.1" iyz="0"
+          izz="0.1"
+      />
+    </inertial>
+  <visual name='left_wheel'>
+      <origin xyz="0 0 0" rpy=" 0 1.5707 1.5707"/>
       <geometry>
-        <cylinder radius='0.1651' length='0.1143'/>
+        <cylinder radius="0.06" length="0.05"/>
+      </geometry>
+      <material name="green"/>
+    </visual>
+  <collision name='left_wheel'>
+      <origin xyz="0 0 0" rpy=" 0 1.5707 1.5707"/>
+      <geometry>
+        <cylinder radius="0.06" length="0.05"/>
       </geometry>
     </collision>
-    <visual>
-      <origin xyz="0 0 0" rpy="0 -0 0"/>
+  </link>
+  <gazebo reference = "left_wheel">
+    <material> Gazebo/Gray </material>
+  </gazebo>
+  <link name="right_wheel">
+  <inertial>
+    <mass value="5.0"/>
+    <origin xyz="0.0 0 0" rpy=" 0 1.5707 1.5707"/>
+    <inertia
+          ixx="0.1" ixy="0" ixz="0"
+          iyy="0.1" iyz="0"
+          izz="0.1"
+      />
+    </inertial>
+  <visual name='right_wheel'>
+      <origin xyz="0 0 0" rpy=" 0 1.5707 1.5707"/>
       <geometry>
-        <mesh filename="package://my_robot/meshes/wheel.dae" scale='0.75 0.75 0.75'/>
+        <cylinder radius="0.06" length="0.05"/>
+      </geometry>
+      <material name="green"/>
+    </visual>
+  <collision name='right_wheel'>
+      <origin xyz="0 0 0" rpy=" 0 1.5707 1.5707"/>
+      <geometry>
+        <cylinder radius="0.06" length="0.05"/>
+      </geometry>
+    </collision>
+  </link>
+  <gazebo reference = "right_wheel">
+    <material> Gazebo/Gray </material>
+  </gazebo>
+  <link name="camera">
+    <box_inertia x="0.05" y="0.05" z="0.05" m="0.1" />
+    <inertial>
+      <mass value="0.1"/>
+      <origin xyz="0.0 0.0 0.0" rpy="0.0 0.0 0.0"/>
+      <inertia ixx="1e-6" ixy="0" ixz="0" iyy="1e-6" iyz="0" izz="1e-6"/>
+    </inertial>
+    <visual name="camera">
+      <origin xyz="0.0 0.0 0.0" rpy="0.0 0.0 0.0"/>
+      <geometry>
+        <box size="0.05 0.05 0.05"/>
+      </geometry>
+      <material name="red"/>
+    </visual>
+    <collision>
+      <origin xyz="0.0 0.0 0.0" rpy="0.0 0.0 0.0"/>
+      <geometry>
+        <box size="0.05 0.05 0.05"/>
+      </geometry>
+    </collision>
+  </link>
+  <gazebo reference = "camera">
+    <material> Gazebo/Red </material>
+  </gazebo>
+  <link name="hokuyo">
+    <inertial>
+      <origin xyz="0.0 0.0 0.0" rpy="0.0 0.0 0.0"/>
+      <mass value="1e-5"/>
+      <inertia ixx="1e-6" ixy="0" ixz="0" iyy="1e-6" iyz="0" izz="1e-6"/>
+    </inertial>
+    <visual name="hokuyo">
+      <origin xyz="0.0 0.0 0.0" rpy="0.0 0.0 0.0"/>
+      <geometry>
+        <mesh filename="package://my_robot/meshes/hokuyo.dae" />
       </geometry>
     </visual>
-    <inertial>
-      <origin xyz='0 0 0' rpy='0 -0 0'/>
-      <mass value='2.637'/>
-      <inertia ixx='0.02467' ixy='0' ixz='0' iyy='0.04411' iyz='0' izz='0.02467'/>
-    </inertial>
-  </link>
-  <link name='front_right_wheel'>
     <collision>
-      <origin xyz='0 0 0' rpy='-1.57079 0 0'/>
+      <origin xyz="0.0 0.0 0.0" rpy="0.0 0.0 0.0"/>
       <geometry>
-        <cylinder radius='0.1651' length='0.1143'/>
+        <box size="0.1 0.1 0.1"/>
       </geometry>
     </collision>
-    <visual>
-      <origin xyz="0 0 0" rpy="0 -0 0"/>
-      <geometry>
-        <mesh filename="package://my_robot/meshes/wheel.dae" scale='0.75 0.75 0.75'/>
-      </geometry>
-    </visual>
-    <inertial>
-      <origin xyz='0 0 0' rpy='0 -0 0'/>
-      <mass value='2.637'/>
-      <inertia ixx='0.02467' ixy='0' ixz='0' iyy='0.04411' iyz='0' izz='0.02467'/>
-    </inertial>
   </link>
-  <link name='back_left_wheel'>
-    <collision>
-      <origin xyz='0 0 0' rpy='-1.57079 0 0'/>
-      <geometry>
-        <cylinder radius='0.1651' length='0.1143'/>
-      </geometry>
-    </collision>
-    <visual>
-      <origin xyz="0 0 0" rpy="0 -0 0"/>
-      <geometry>
-        <mesh filename="package://my_robot/meshes/wheel.dae" scale='0.75 0.75 0.75'/>
-      </geometry>
-    </visual>
-    <inertial>
-      <origin xyz='0 0 0' rpy='0 -0 0'/>
-      <mass value='2.637'/>
-      <inertia ixx='0.02467' ixy='0' ixz='0' iyy='0.04411' iyz='0' izz='0.02467'/>
-    </inertial>
-  </link>
-  <link name='back_right_wheel'>
-    <collision>
-      <origin xyz='0 0 0' rpy='-1.57079 0 0'/>
-      <geometry>
-        <cylinder radius='0.1651' length='0.1143'/>
-      </geometry>
-    </collision>
-    <visual>
-      <origin xyz="0 0 0" rpy="0 -0 0"/>
-      <geometry>
-        <mesh filename="package://my_robot/meshes/wheel.dae" scale='0.75 0.75 0.75'/>
-      </geometry>
-    </visual>
-    <inertial>
-      <origin xyz='0 0 0' rpy='0 -0 0'/>
-      <mass value='2.637'/>
-      <inertia ixx='0.02467' ixy='0' ixz='0' iyy='0.04411' iyz='0' izz='0.02467'/>
-    </inertial>
-  </link>
-  <joint type="continuous" name="front_left_wheel_hinge">
-    <origin xyz="0.2 0.25 0" rpy="0 0 0"/>
-    <child link="front_left_wheel"/>
+  <joint type="continuous" name="left_wheel_hinge">
+    <origin xyz="0 0.1 -0.04" rpy="0 0 0"/>
+    <child link="left_wheel"/>
     <parent link="chassis"/>
     <axis xyz="0 1 0" rpy="0 0 0"/>
@@ -116,7 +160,7 @@
     <dynamics damping="1.0" friction="1.0"/>
   </joint>
-  <joint type="continuous" name="front_right_wheel_hinge">
-    <origin xyz="0.2 -0.25 0" rpy="0 0 0"/>
-    <child link="front_right_wheel"/>
+  <joint type="continuous" name="right_wheel_hinge">
+    <origin xyz="0 -0.1 -0.04" rpy="0 0 0"/>
+    <child link="right_wheel"/>
     <parent link="chassis"/>
     <axis xyz="0 1 0" rpy="0 0 0"/>
@@ -124,90 +168,19 @@
     <dynamics damping="1.0" friction="1.0"/>
   </joint>
-  <joint type="continuous" name="rear_left_wheel_hinge">
-    <origin xyz="-0.2 0.255555 0" rpy="0 0 0"/>
-    <child link="back_left_wheel"/>
+  <joint name="robot_footprint_joint" type="fixed">
+    <origin xyz="0 0 0" rpy="0 0 0" />
+    <parent link="robot_footprint"/>
+    <child link="chassis" />
+  </joint>
+  <joint name="camera_name" type="fixed">
+   <origin xyz="0.15 0.0 0.0" rpy="0.0 0.0 0.0"/>
+   <parent link="chassis"/>
+   <child link="camera"/>
+   <axis xyz="0 1 0"/>
+  </joint>
+  <joint name="hokuyo_joint" type="fixed">
+    <origin xyz="0.1 0.0 0.1" rpy="0.0 0.0 0.0"/>
     <parent link="chassis"/>
-    <axis xyz="0 1 0" rpy="0 0 0"/>
-    <limit effort="10000" velocity="1000"/>
-    <dynamics damping="1.0" friction="1.0"/>
+    <child link="hokuyo"/>
   </joint>
-  <joint type="continuous" name="rear_right_wheel_hinge">
-    <origin xyz="-0.2 -0.25 0" rpy="0 0 0"/>
-    <child link="back_right_wheel"/>
-    <parent link="chassis"/>
-    <axis xyz="0 1 0" rpy="0 0 0"/>
-    <limit effort="10000" velocity="1000"/>
-    <dynamics damping="1.0" friction="1.0"/>
-  </joint>
-  <link name="camera">
-    <inertial>
-      <mass value="0.1" />
-      <origin xyz="0 0 0" rpy="0 0 0" />
-      <box_inertia m="0.1" x="0.05" y="0.05" z="0.05"/>
-      <inertia
-        ixx="1e-6" ixy="0" ixz="0"
-        iyy="1e-6" iyz="0"
-        izz="1e-6"
-      />
-    </inertial>
-    <collision>
-      <origin xyz="0 0 0" rpy="0 0 0" />
-      <geometry>
-        <box  size="0.05 0.05 0.05"/>
-      </geometry>
-    </collision>
-    <visual>
-     <origin xyz="0 0 0" rpy="0 0 0" />
-      <geometry>
-        <mesh filename="package://my_robot/meshes/realsense.dae" />
-      </geometry>
-    </visual>
-  </link>
-  <joint type="fixed" name="camera_joint">
-    <axis xyz="0 1 0"/>
-    <origin xyz="0.25 0 0" rpy="0 0 0" />
-    <parent link="chassis" />
-    <child link="camera" />
-  </joint>
-  <link name="hokuyo">
-    <inertial>
-      <mass value="1e-5" />
-      <origin xyz="0 0 0" rpy="0 0 0" />
-      <inertia
-        ixx="1e-6" ixy="0" ixz="0"
-        iyy="1e-6" iyz="0"
-        izz="1e-6"
-      />
-    </inertial>
-    <collision>
-      <origin xyz="0 0 0" rpy="0 0 0" />
-      <geometry>
-        <box  size="0.1 0.1 0.1"/>
-      </geometry>
-    </collision>
-    <visual>
-      <origin xyz="0 0 0" rpy="0 0 0" />
-      <geometry>
-        <mesh filename="package://my_robot/meshes/hokuyo.dae" />
-      </geometry>
-    </visual>
-  </link>
-  <joint type="fixed" name="hokuyo_joint">
-    <axis xyz="0 1 0"/>
-    <origin xyz="0 0 0.14" rpy="0 0 0" />
-    <parent link="chassis" />
-    <child link="hokuyo" />
-  </joint>
-  <!--<gazebo reference="left_wheel">
-    <material>Gazebo/Black</material>
-  </gazebo>
-  <gazebo reference="right_wheel">
-    <material>Gazebo/Black</material>
-  </gazebo>
-  <gazebo reference="camera">
-    <material>Gazebo/Grey</material>
-  </gazebo>-->
-  <gazebo reference="chassis">
-    <material>Gazebo/Green</material>
-  </gazebo>
 </robot>
